Commit message: Add adaptive gripper simulation model

File: models/puppybot/final2/urdf/final2.urdf (robot description, URDF)
Before this commit: robot final2, 221 links, 220 joints
Links:
- added link gripper_base; visual mesh filename=package://final2/meshes/adaptive_gripper/gripper_base.gltf scale=1 1 1
- added link gripper_left1; visual mesh filename=package://final2/meshes/adaptive_gripper/gripper_left1.gltf scale=1 1 1
- added link gripper_left2; visual mesh filename=package://final2/meshes/adaptive_gripper/gripper_left2.gltf scale=1 1 1
- added link gripper_left3; visual mesh filename=package://final2/meshes/adaptive_gripper/gripper_left3.gltf scale=1 1 1
- added link gripper_right1; visual mesh filename=package://final2/meshes/adaptive_gripper/gripper_right1.gltf scale=1 1 1
- added link gripper_right2; visual mesh filename=package://final2/meshes/adaptive_gripper/gripper_right2.gltf scale=1 1 1
- added link gripper_right3; visual mesh filename=package://final2/meshes/adaptive_gripper/gripper_right3.gltf scale=1 1 1
Joints:
- added joint gripper_base_to_gripper_left2: type revolute, parent gripper_base, child gripper_left2, origin xyz=-0.005 0.027 0 rpy=0 0 0, axis 0 0 1, limit lower=-0.8 upper=0.5 effort=1000 velocity=2
- added joint gripper_base_to_gripper_right2: type revolute, parent gripper_base, child gripper_right2, origin xyz=0.005 0.027 0 rpy=0 0 0, axis 0 0 1, limit lower=-0.5 upper=0.8 effort=1000 velocity=2
- added joint gripper_base_to_gripper_right3: type revolute, parent gripper_base, child gripper_right3, origin xyz=0.012 0.005 0 rpy=0 0 0, axis 0 0 1, limit lower=-0.15 upper=0.7 effort=1000 velocity=2
- added joint gripper_controller: type revolute, parent gripper_base, child gripper_left3, origin xyz=-0.012 0.005 0 rpy=0 0 0, axis 0 0 1, limit lower=-0.7 upper=0.15 effort=1000 velocity=2
- added joint gripper_left3_to_gripper_left1: type revolute, parent gripper_left3, child gripper_left1, origin xyz=-0.027 0.016 0 rpy=0 0 0, axis 0 0 1, limit lower=-0.5 upper=0.5 effort=1000 velocity=2
- added joint gripper_right3_to_gripper_right1: type revolute, parent gripper_right3, child gripper_right1, origin xyz=0.027 0.016 0 rpy=0 0 0, axis 0 0 1, limit lower=-0.5 upper=0.5 effort=1000 velocity=2
- added joint part_1_4_to_gripper_base: type fixed, parent part_1_4, child gripper_base, origin xyz=0.0383 0 -0.045 rpy=0.866 0 1.5708

Commit message: Align adaptive gripper with TCP forward axis

File: models/puppybot/final2/urdf/final2.urdf (robot description, URDF)
Before this commit: robot final2, 228 links, 227 joints
Joints:
- joint part_1_4_to_gripper_base: origin xyz=0.0383 0 -0.045 rpy=0.866 0 1.5708 -> xyz=0.0383 0 -0.045 rpy=0 0 1.5708

Commit message: Mount adaptive gripper by its rear flange

File: models/puppybot/final2/urdf/final2.urdf (robot description, URDF)
Before this commit: robot final2, 228 links, 227 joints
Joints:
- joint part_1_4_to_gripper_base: origin xyz=0.0383 0 -0.045 rpy=0 0 1.5708 -> xyz=0.0723 0 -0.045 rpy=0 0 -1.5708

Commit message: Point adaptive gripper upward

File: models/puppybot/final2/urdf/final2.urdf (robot description, URDF)
Before this commit: robot final2, 228 links, 227 joints
Joints:
- joint part_1_4_to_gripper_base: origin xyz=0.0723 0 -0.045 rpy=0 0 -1.5708 -> xyz=0.0383 0 -0.079 rpy=-1.5708 0 0

Commit message: Center gripper on wrist flange

File: models/puppybot/final2/urdf/final2.urdf (robot description, URDF)
Before this commit: robot final2, 228 links, 227 joints
Joints:
- joint part_1_4_to_gripper_base: origin xyz=0.0383 0 -0.079 rpy=-1.5708 0 0 -> xyz=0.038 -0.00185 -0.03932 rpy=-1.5708 0 0

Commit message: Integrate gripper support and runtime logging
Add configurable gripper speed, feedback telemetry, status safety
handling, and
RobotDreams virtual-servo wiring. Document log-file selection and update
scenario settling for optional gripper state.

File: models/puppybot/final2/urdf/final2.urdf (robot description, URDF)
Before this commit: robot final2, 228 links, 227 joints
Joints:
- joint part_1_4_to_gripper_base: origin xyz=0.038 -0.00185 -0.03932 rpy=-1.5708 0 0 -> xyz=0.018 -0.0022 -0.06932 rpy=-1.5708 0 0
